Commit message: urdf/matilda_macro.xacro: fix visual for link_1
fixes #1

File: urdf/matilda_macro.xacro (robot description, xacro)
@@ -24,5 +24,5 @@
 	<link name="${prefix}link_1">
 		<visual>
-			<origin xyz="-0.2 0 0" rpy="0 0 0"/>
+			<origin xyz="0 0 0" rpy="0 0 0"/>
 			<geometry>
 				<mesh filename="package://matilda_support/meshes/link_1.stl"/>

Commit message: urdf/matilda_macro.xacro: add dummy joints for cartesian planning

File: urdf/matilda_macro.xacro (robot description, xacro)
@@ -117,4 +117,6 @@
 	</link>
 	<link name="${prefix}tool0"/>
+	<link name="${prefix}dummy_1"/>
+	<link name="${prefix}dummy_2"/>
 	<!-- end of link list -->
 	<!-- joint list -->
@@ -152,4 +154,16 @@
 		<origin xyz="0 0 0" rpy="0 1.57079632679 0"/>
 	</joint>
+	<joint name="${prefix}dummy_1" type="continuous">
+		<parent link="${prefix}tool0"/>
+		<child link="${prefix}dummy_1"/>
+		<axis xyz="1 0 0"/>
+		<origin xyz="0 0 0" rpy="0 -1.57079632679 0"/>
+	</joint>
+	<joint name="${prefix}dummy_2" type="continuous">
+		<parent link="${prefix}dummy_1"/>
+		<child link="${prefix}dummy_2"/>
+		<axis xyz="0 0 1"/>
+		<origin xyz="0 0 0" rpy="0 0 0"/>
+	</joint>
 	<!-- end of joint list -->
 	<!-- ROS base_link to Matilda World Coordinates transform -->

Commit message: matilda_macro.xacro: fix world tf

File: urdf/matilda_macro.xacro (robot description, xacro)
@@ -157,6 +157,6 @@
 	<joint name="${prefix}base_link-base" type="fixed">
 		<origin xyz="0 0 0" rpy="0 0 0"/>
-		<parent link="${prefix}base_link"/>
-		<child link="${prefix}base"/>
+		<parent link="${prefix}base"/>
+		<child link="${prefix}base_link"/>
 	</joint>
 </xacro:macro>

Commit message: matilda_xacro: update link names

File: urdf/matilda_macro.xacro (robot description, xacro)
@@ -117,6 +117,6 @@
 	</link>
 	<link name="${prefix}tool0"/>
-	<link name="${prefix}dummy_1"/>
-	<link name="${prefix}dummy_2"/>
+	<link name="${prefix}link_5"/>
+	<link name="${prefix}link_6"/>
 	<!-- end of link list -->
 	<!-- joint list -->
@@ -154,13 +154,13 @@
 		<origin xyz="0 0 0" rpy="0 1.57079632679 0"/>
 	</joint>
-	<joint name="${prefix}dummy_1" type="continuous">
+	<joint name="${prefix}joint_5" type="continuous">
 		<parent link="${prefix}tool0"/>
-		<child link="${prefix}dummy_1"/>
+		<child link="${prefix}link_5"/>
 		<axis xyz="1 0 0"/>
 		<origin xyz="0 0 0" rpy="0 -1.57079632679 0"/>
 	</joint>
-	<joint name="${prefix}dummy_2" type="continuous">
-		<parent link="${prefix}dummy_1"/>
-		<child link="${prefix}dummy_2"/>
+	<joint name="${prefix}joint_6" type="continuous">
+		<parent link="${prefix}link_5"/>
+		<child link="${prefix}link_6"/>
 		<axis xyz="0 0 1"/>
 		<origin xyz="0 0 0" rpy="0 0 0"/>
