Commit message: add correct limits and velocities

File: urdf/matilda.URDF (robot description, URDF)
Before this commit: robot matilda_support, 8 links, 7 joints
Joints:
- joint joint_1: limit lower=-2 upper=2 effort=0 velocity=0 -> lower=-2 upper=2 effort=0 velocity=1.57079632679
- joint joint_2: limit lower=-0.8 upper=2.5 effort=0 velocity=0 -> lower=-0.75 upper=2.5 effort=0 velocity=1.57079632679
- joint joint_3: limit lower=-0.8 upper=1.7 effort=0 velocity=0 -> lower=-1.4 upper=1.57079632679 effort=0 velocity=1.57079632679
- joint joint_4: limit lower=-3.2 upper=3.2 effort=0 velocity=0 -> lower=-3.2 upper=3.2 effort=0 velocity=1.57079632679
- joint joint_5: limit lower=-1.8 upper=1.8 effort=0 velocity=0 -> lower=-1.57079632679 upper=1.57079632679 effort=0 velocity=1.57079632679

File: urdf/matilda_macro.xacro (robot description, xacro)
@@ -125,5 +125,5 @@
 		<child link="link_1" />
 		<axis xyz="0 0 -1" />
-		<limit lower="-2" upper="2" effort="0" velocity="0" />
+		<limit lower="-2" upper="2" effort="0" velocity="1.57079632679" />
 	</joint>
 	<joint name="${prefix}joint_2" type="revolute">
@@ -132,5 +132,5 @@
 		<child link="${prefix}link_2"/>
 		<axis xyz="0 1 0"/>
-		<limit lower="-0.8" upper="2.5" effort="0" velocity="0"/>
+		<limit lower="-0.75" upper="2.5" effort="0" velocity="1.57079632679"/>
 	</joint>
 	<joint name="${prefix}joint_3" type="revolute">
@@ -139,5 +139,5 @@
 		<child link="${prefix}link_3"/>
 		<axis xyz="0 -1 0"/>
-		<limit lower="-0.8" upper="1.7" effort="0" velocity="0"/>
+		<limit lower="-1.4" upper="1.57079632679" effort="0" velocity="1.57079632679"/>
 	</joint>
 	<joint name="${prefix}joint_4" type="revolute">
@@ -146,5 +146,5 @@
 		<child link="${prefix}link_4"/>
 		<axis xyz="0.99737 0 -0.072536"/>
-		<limit lower="-3.2" upper="3.2" effort="0" velocity="0"/>
+		<limit lower="-3.2" upper="3.2" effort="0" velocity="1.57079632679"/>
 	</joint>
 	<joint name="${prefix}joint_5" type="revolute">
@@ -153,5 +153,5 @@
 		<child link="${prefix}link_5"/>
 		<axis xyz="0 1 0"/>
-		<limit lower="-1.8" upper="1.8" effort="0" velocity="0"/>
+		<limit lower="-1.57079632679" upper="1.57079632679" effort="0" velocity="1.57079632679"/>
 	</joint>
 	<joint name="${prefix}joint_5-tool0" type="fixed">

Commit message: urdf: change updated geometry

File: urdf/matilda.URDF (robot description, URDF)
Before this commit: robot matilda_support, 8 links, 7 joints
Joints:
- joint joint_1: origin xyz=0 0 0.037 rpy=0 0 0 -> xyz=0 0 0.103 rpy=0 0 0

File: urdf/matilda_macro.xacro (robot description, xacro)
@@ -24,5 +24,5 @@
 	<link name="${prefix}link_1">
 		<visual>
-			<origin xyz="0 0 0" rpy="0 0 0"/>
+			<origin xyz="-0.2 0 0" rpy="0 0 0"/>
 			<geometry>
 				<mesh filename="package://matilda_support/meshes/link_1.STL"/>
@@ -121,5 +121,5 @@
 	<!-- joint list -->
 	<joint name="${prefix}joint_1" type="revolute">
-		<origin xyz="0 0 0.037" rpy="0 0 0" />
+		<origin xyz="0 0 0.103" rpy="0 0 0" />
 		<parent link="base_link" />
 		<child link="link_1" />

Commit message: fix wrist joint

File: urdf/matilda.URDF (robot description, URDF)
Before this commit: robot matilda_support, 8 links, 7 joints
Joints:
- joint joint_4: limit lower=-3.2 upper=3.2 effort=0 velocity=1.57079632679 -> (none); type revolute -> fixed

File: urdf/matilda_macro.xacro (robot description, xacro)
@@ -141,10 +141,10 @@
 		<limit lower="-1.4" upper="1.57079632679" effort="0" velocity="1.57079632679"/>
 	</joint>
-	<joint name="${prefix}joint_4" type="revolute">
+	<joint name="${prefix}joint_4" type="fixed">
 		<origin xyz="0.18 0 0.027015" rpy="0 0 0"/>
 		<parent link="${prefix}link_3"/>
 		<child link="${prefix}link_4"/>
 		<axis xyz="0.99737 0 -0.072536"/>
-		<limit lower="-3.2" upper="3.2" effort="0" velocity="1.57079632679"/>
+		<!-- <limit lower="-3.2" upper="3.2" effort="0" velocity="1.57079632679"/> -->
 	</joint>
 	<joint name="${prefix}joint_5" type="revolute">

Commit message: Lowercase file extensions.

File: urdf/matilda.URDF (robot description, URDF)
Before this commit: robot matilda_support, 8 links, 7 joints
Links:
- link base_link: geometry collision mesh filename=package://matilda_support/meshes/base_link.stl; visual mesh filename=package://matilda_support/meshes/base_link.stl
- link link_1: geometry collision mesh filename=package://matilda_support/meshes/link_1.stl; visual mesh filename=package://matilda_support/meshes/link_1.stl
- link link_2: geometry collision mesh filename=package://matilda_support/meshes/link_2.stl; visual mesh filename=package://matilda_support/meshes/link_2.stl
- link link_3: geometry collision mesh filename=package://matilda_support/meshes/link_3.stl; visual mesh filename=package://matilda_support/meshes/link_3.stl
- link link_4: geometry collision mesh filename=package://matilda_support/meshes/link_4.stl; visual mesh filename=package://matilda_support/meshes/link_4.stl
- link link_5: geometry collision mesh filename=package://matilda_support/meshes/link_5.stl; visual mesh filename=package://matilda_support/meshes/link_5.stl

File: urdf/matilda_macro.xacro (robot description, xacro)
@@ -7,5 +7,5 @@
 			<origin xyz="0 0 0" rpy="0 0 0"/>
 			<geometry>
-				<mesh filename="package://matilda_support/meshes/base_link.STL"/>
+				<mesh filename="package://matilda_support/meshes/base_link.stl"/>
 			</geometry>
 			<material name="matilda_grey">
@@ -15,5 +15,5 @@
 		<collision>
 			<geometry>
-				<mesh filename="package://matilda_support/meshes/base_link.STL"/>
+				<mesh filename="package://matilda_support/meshes/base_link.stl"/>
 			</geometry>
 			<material name="red">
@@ -26,5 +26,5 @@
 			<origin xyz="-0.2 0 0" rpy="0 0 0"/>
 			<geometry>
-				<mesh filename="package://matilda_support/meshes/link_1.STL"/>
+				<mesh filename="package://matilda_support/meshes/link_1.stl"/>
 			</geometry>
 			<material name="matilda_grey">
@@ -34,5 +34,5 @@
 		<collision>
 			<geometry>
-				<mesh filename="package://matilda_support/meshes/link_1.STL"/>
+				<mesh filename="package://matilda_support/meshes/link_1.stl"/>
 			</geometry>
 			<material name="red">
@@ -45,5 +45,5 @@
 			<origin xyz="0 0 0" rpy="0 0 0"/>
 			<geometry>
-				<mesh filename="package://matilda_support/meshes/link_2.STL"/>
+				<mesh filename="package://matilda_support/meshes/link_2.stl"/>
 			</geometry>
 			<material name="matilda_grey">
@@ -53,5 +53,5 @@
 		<collision>
 			<geometry>
-				<mesh filename="package://matilda_support/meshes/link_2.STL"/>
+				<mesh filename="package://matilda_support/meshes/link_2.stl"/>
 			</geometry>
 			<material name="red">
@@ -64,5 +64,5 @@
 			<origin xyz="0 0 0" rpy="0 0 0"/>
 			<geometry>
-				<mesh filename="package://matilda_support/meshes/link_3.STL"/>
+				<mesh filename="package://matilda_support/meshes/link_3.stl"/>
 			</geometry>
 			<material name="matilda_grey">
@@ -72,5 +72,5 @@
 		<collision>
 			<geometry>
-				<mesh filename="package://matilda_support/meshes/link_3.STL"/>
+				<mesh filename="package://matilda_support/meshes/link_3.stl"/>
 			</geometry>
 			<material name="red">
@@ -83,5 +83,5 @@
 			<origin xyz="0 0 0" rpy="0 0 0"/>
 			<geometry>
-				<mesh filename="package://matilda_support/meshes/link_4.STL"/>
+				<mesh filename="package://matilda_support/meshes/link_4.stl"/>
 			</geometry>
 			<material name="matilda_grey">
@@ -91,5 +91,5 @@
 		<collision>
 			<geometry>
-				<mesh filename="package://matilda_support/meshes/link_4.STL"/>
+				<mesh filename="package://matilda_support/meshes/link_4.stl"/>
 			</geometry>
 			<material name="red">
@@ -102,5 +102,5 @@
 			<origin xyz="0 0 0" rpy="0 0 0"/>
 			<geometry>
-				<mesh filename="package://matilda_support/meshes/link_5.STL"/>
+				<mesh filename="package://matilda_support/meshes/link_5.stl"/>
 			</geometry>
 			<material name="matilda_grey">
@@ -110,5 +110,5 @@
 		<collision>
 			<geometry>
-				<mesh filename="package://matilda_support/meshes/link_5.STL"/>
+				<mesh filename="package://matilda_support/meshes/link_5.stl"/>
 			</geometry>
 			<material name="red">

Commit message: urdf: remove wrist joint cleanup

File: urdf/matilda.URDF (robot description, URDF)
Before this commit: robot matilda_support, 8 links, 7 joints
Links:
- removed link link_5
- link link_3: geometry collision mesh filename=package://matilda_support/meshes/link_3.stl; collision mesh filename=package://matilda_support/meshes/link_4_old.stl
Joints:
- removed joint joint_5
- removed joint joint_5-tool0
- added joint joint_4-tool0: type fixed, parent link_4, child tool0, origin xyz=0 0 0 rpy=0 1.57079632679 0
- joint joint_4: axis 0.99737 0 -0.072536 -> 0 1 0; limit (none) -> lower=-1.57079632679 upper=1.57079632679 effort=0 velocity=1.57079632679; origin xyz=0.18 0 0.027015 rpy=0 0 0 -> xyz=0.55145 0 0 rpy=0 0 0; type fixed -> revolute

File: urdf/matilda_macro.xacro (robot description, xacro)
@@ -70,4 +70,13 @@
 			</material>
 		</visual>
+		<visual>
+			<origin xyz="0.18 0 0.027015" rpy="0 0 0"/>
+			<geometry>
+				<mesh filename="package://matilda_support/meshes/link_4_old.stl"/>
+			</geometry>
+			<material name="matilda_grey">
+				<color rgba="0.5 0.5 0.5 1"/>
+			</material>
+		</visual>
 		<collision>
 			<geometry>
@@ -76,4 +85,13 @@
 			<material name="red">
 				<color rgba="1 0 0 1"/>
+			</material>
+		</collision>
+		<collision>
+			<origin xyz="0.18 0 0.027015" rpy="0 0 0"/>
+			<geometry>
+				<mesh filename="package://matilda_support/meshes/link_4_old.stl"/>
+			</geometry>
+			<material name="red">
+				<color rgba="0.5 0.5 0.5 1"/>
 			</material>
 		</collision>
@@ -92,23 +110,4 @@
 			<geometry>
 				<mesh filename="package://matilda_support/meshes/link_4.stl"/>
-			</geometry>
-			<material name="red">
-				<color rgba="1 0 0 1"/>
-			</material>
-		</collision>
-	</link>
-	<link name="${prefix}link_5">
-		<visual>
-			<origin xyz="0 0 0" rpy="0 0 0"/>
-			<geometry>
-				<mesh filename="package://matilda_support/meshes/link_5.stl"/>
-			</geometry>
-			<material name="matilda_grey">
-				<color rgba="0.5 0.5 0.5 1"/>
-			</material>
-		</visual>
-		<collision>
-			<geometry>
-				<mesh filename="package://matilda_support/meshes/link_5.stl"/>
 			</geometry>
 			<material name="red">
@@ -141,20 +140,13 @@
 		<limit lower="-1.4" upper="1.57079632679" effort="0" velocity="1.57079632679"/>
 	</joint>
-	<joint name="${prefix}joint_4" type="fixed">
-		<origin xyz="0.18 0 0.027015" rpy="0 0 0"/>
+	<joint name="${prefix}joint_4" type="revolute">
+		<origin xyz="0.55145 0 0" rpy="0 0 0"/>
 		<parent link="${prefix}link_3"/>
 		<child link="${prefix}link_4"/>
-		<axis xyz="0.99737 0 -0.072536"/>
-		<!-- <limit lower="-3.2" upper="3.2" effort="0" velocity="1.57079632679"/> -->
-	</joint>
-	<joint name="${prefix}joint_5" type="revolute">
-		<origin xyz="0.37145 0 -0.0270150" rpy="0 0 0"/>
-		<parent link="${prefix}link_4"/>
-		<child link="${prefix}link_5"/>
 		<axis xyz="0 1 0"/>
 		<limit lower="-1.57079632679" upper="1.57079632679" effort="0" velocity="1.57079632679"/>
 	</joint>
-	<joint name="${prefix}joint_5-tool0" type="fixed">
-		<parent link="${prefix}link_5"/>
+	<joint name="${prefix}joint_4-tool0" type="fixed">
+		<parent link="${prefix}link_4"/>
 		<child link="${prefix}tool0"/>
 		<origin xyz="0 0 0" rpy="0 1.57079632679 0"/>

Commit message: add generated urdf file for historical purposes

File: urdf/matilda.URDF (robot description, URDF)
Before this commit: robot matilda_support, 7 links, 6 joints
Links:
- added link link_5
- added link link_6
Joints:
- added joint joint_5: type continuous, parent tool0, child link_5, origin xyz=0 0 0 rpy=0 -1.57079632679 0, axis 1 0 0
- added joint joint_6: type continuous, parent link_5, child link_6, origin xyz=0 0 0 rpy=0 0 0, axis 0 0 1
